Commit message: Fix end effecto offset

File: pm_grasp_visualization/launch/uwsim/gripper_for_spec.urdf (robot description, URDF)
Before this commit: robot arm5e_gripper, 4 links, 3 joints
Links:
- added link base_link
Joints:
- added joint base_link_to_part4_base: type fixed, parent base_link, child part4_base, origin xyz=0 0 -0.1485 rpy=0 0 0
- joint JawOpening: axis 1 0 0 -> 0 -1 0; origin xyz=0 -0.04 0.045 rpy=0 0 0 -> xyz=-0.04 0 0.045 rpy=0 0 0
- joint part4_to_link4_jaw2: axis -1 0 0 -> 0 1 0; origin xyz=0 0.04 0.0450 rpy=0 0 0 -> xyz=0.04 0 0.0450 rpy=0 0 0
