Commit message: Change position of UWSim stuff

File: pm_grasp_visualization/launch/uwsim/data/scenes/cloud_source.urdf (robot description, URDF)
Before this commit: robot cloud_source, 3 links, 2 joints
Links:
- added link camera
Joints:
- added joint base_to_uib_camera: type fixed, parent base_link, child camera, origin xyz=0 0 0 rpy=0 0 0
