Commit message: Add STL files to URDF for RViz

File: pm_manipulation/launch/arm5e_with_sensor.urdf (robot description, URDF)
Before this commit: robot arm5e, 10 links, 9 joints
Links:
- link part1: geometry visual mesh filename=package://pm_manipulation/launch/uwsim/data/robot/ARM5E/ARM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
- link part2: geometry visual mesh filename=package://pm_manipulation/launch/uwsim/data/robot/ARM5E/ARM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
- link part3: geometry visual mesh filename=package://pm_manipulation/launch/uwsim/data/robot/ARM5E/ARM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
- link part4_base: geometry visual mesh filename=package://pm_manipulation/launch/uwsim/data/robot/ARM5E/ARM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
- link part4_jaw1: geometry visual mesh filename=package://pm_manipulation/launch/uwsim/data/robot/ARM5E/ARM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
- link part4_jaw2: geometry visual mesh filename=package://pm_manipulation/launch/uwsim/data/robot/ARM5E/ARM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
